Commit message: Updated URDF to put end effector geometry into sand_tcp link

File: urdf/workcell.xacro (robot description, xacro)
@@ -113,9 +113,4 @@
       </geometry>
     </visual>
-    <visual>
-      <geometry>
-        <mesh filename="package://snp_automate_2023/meshes/collision/sponge.ply"/>
-      </geometry>
-    </visual>
     <!-- Collision -->
     <collision>
@@ -154,9 +149,4 @@
       </geometry>
     </collision>
-    <collision>
-      <geometry>
-        <mesh filename="package://snp_automate_2023/meshes/collision/sponge.ply"/>
-      </geometry>
-    </collision>
   </link>
   <joint name="tool0_to_ee" type="fixed">
@@ -187,5 +177,16 @@
   </joint>
   <!-- Add TCP -->
-  <link name="sand_tcp"/>
+  <link name="sand_tcp">
+    <visual>
+      <geometry>
+        <mesh filename="package://snp_automate_2023/meshes/collision/sponge.ply"/>
+      </geometry>
+    </visual>
+    <collision>
+      <geometry>
+        <mesh filename="package://snp_automate_2023/meshes/collision/sponge.ply"/>
+      </geometry>
+    </collision>
+  </link>
   <joint name="sand_tcp_joint" type="fixed">
     <parent link="tool_flange"/>

Commit message: Removed TCP geometry

File: urdf/workcell.xacro (robot description, xacro)
@@ -178,12 +178,16 @@
   <!-- Add TCP -->
   <link name="sand_tcp">
-    <visual>
-      <geometry>
-        <mesh filename="package://snp_automate_2023/meshes/collision/sponge.ply"/>
-      </geometry>
-    </visual>
-    <collision>
-      <geometry>
-        <mesh filename="package://snp_automate_2023/meshes/collision/sponge.ply"/>
+<!--    <visual>-->
+<!--      <origin xyz="0 0 -0.0325" />-->
+<!--      <geometry>-->
+<!--        <cylinder radius="0.030" length="0.025"/>-->
+<!--        <mesh filename="package://snp_automate_2023/meshes/collision/sponge.ply"/>-->
+<!--      </geometry>-->
+<!--    </visual>-->
+    <collision>
+      <origin xyz="0 0 -0.0325" />
+      <geometry>
+        <cylinder radius="0.030" length="0.025"/>
+<!--        <mesh filename="package://snp_automate_2023/meshes/collision/sponge.ply"/>-->
       </geometry>
     </collision>
@@ -192,5 +196,5 @@
     <parent link="tool_flange"/>
 <!--    <origin xyz="-0.158 -0.158 0.123" rpy="0.0 ${radians(90)} ${radians(-135)}"/>-->
-    <origin xyz="-0.149 ${-0.149 - 0.005} 0.123" rpy="0.0 ${radians(90)} ${radians(-135)}"/>
+    <origin xyz="-0.149 ${-0.149 - 0.020} 0.123" rpy="0.0 ${radians(90)} ${radians(-135)}"/>
 <!--    <parent link="ee"/>-->
 <!--    <origin xyz="${-0.186 - 0.038} 0.0 ${0.08325}" rpy="0.0 ${radians(90)} 0.0"/>-->

Commit message: Added camera TCP

File: urdf/workcell.xacro (robot description, xacro)
@@ -176,4 +176,10 @@
             rpy="${camera_cal['target_mount_to_target_rpy']['x']} ${camera_cal['target_mount_to_target_rpy']['y']} ${camera_cal['target_mount_to_target_rpy']['z']}" />
   </joint>
+  <link name="camera_tcp" />
+  <joint name="camera_tcp_joint" type="fixed">
+    <parent link="camera_color_optical_frame"/>
+    <child link="camera_tcp"/>
+    <origin xyz="0 0 0.150" rpy="0 0 0"/>
+  </joint>
   <!-- Add TCP -->
   <link name="sand_tcp">

Commit message: Rotated TCP 180 degrees to accommodate change to SNP motion planning

File: urdf/workcell.xacro (robot description, xacro)
@@ -192,5 +192,5 @@
     <parent link="tool_flange"/>
 <!--    <origin xyz="-0.158 -0.158 0.123" rpy="0.0 ${radians(90)} ${radians(-135)}"/>-->
-    <origin xyz="-0.149 ${-0.149 - 0.005} 0.123" rpy="0.0 ${radians(90)} ${radians(-135)}"/>
+    <origin xyz="-0.149 ${-0.149 - 0.005} 0.123" rpy="0.0 ${radians(-90)} ${radians(-135)}"/>
 <!--    <parent link="ee"/>-->
 <!--    <origin xyz="${-0.186 - 0.038} 0.0 ${0.08325}" rpy="0.0 ${radians(90)} 0.0"/>-->

Commit message: Updated application to specify camera frame relative robot controller-published flange frame

File: urdf/workcell.xacro (robot description, xacro)
@@ -5,5 +5,4 @@
   <xacro:include filename="$(find snp_automate_2023)/urdf/ros2_control.xacro"/>
   <xacro:snp_ros2_control name="snp_ros2_control" prefix=""/>
-  <xacro:property name="dt_flange_width" value="0.040"/>
   <!-- Add World -->
   <material name="light_gray">
@@ -64,11 +63,4 @@
     <child link="base_link"/>
     <origin xyz="-0.61 0 0.723" rpy="0 0 0"/>
-  </joint>
-  <!-- Create a frame representing the robot tool flange (behind the teach tool and nominal tool0 frame) for IKFast -->
-  <link name="tool_flange"/>
-  <joint name="tool0_to_tool_flange" type="fixed">
-    <parent link="tool0"/>
-    <child link="tool_flange"/>
-    <origin xyz="0.0 0.0 ${-dt_flange_width}" rpy="0 0 0"/>
   </joint>
   <!-- Add End Effector Components -->
@@ -162,17 +154,10 @@
     <xacro:property name="camera_cal" value="${load_yaml('$(find snp_automate_2023)/config/calibration.yaml')}" />
   </xacro:unless>
-  <link name="camera_color_optical_frame"/>
+  <link name="camera_frame"/>
   <joint name="tool0_to_camera" type="fixed">
-    <parent link="tool0"/>
-    <child link="camera_color_optical_frame"/>
+    <parent link="flange"/>
+    <child link="camera_frame"/>
     <origin xyz="${camera_cal['camera_mount_to_camera_pos']['x']} ${camera_cal['camera_mount_to_camera_pos']['y']} ${camera_cal['camera_mount_to_camera_pos']['z']}"
             rpy="${camera_cal['camera_mount_to_camera_rpy']['x']} ${camera_cal['camera_mount_to_camera_rpy']['y']} ${camera_cal['camera_mount_to_camera_rpy']['z']}" />
-  </joint>
-  <link name="cal_target_frame"/>
-  <joint name="target_mount_to_target" type="fixed">
-    <parent link="base_link"/>
-    <child link="cal_target_frame"/>
-    <origin xyz="${camera_cal['target_mount_to_target_pos']['x']} ${camera_cal['target_mount_to_target_pos']['y']} ${camera_cal['target_mount_to_target_pos']['z']}"
-            rpy="${camera_cal['target_mount_to_target_rpy']['x']} ${camera_cal['target_mount_to_target_rpy']['y']} ${camera_cal['target_mount_to_target_rpy']['z']}" />
   </joint>
   <!-- Add TCP -->
@@ -190,7 +175,7 @@
   </link>
   <joint name="sand_tcp_joint" type="fixed">
-    <parent link="tool_flange"/>
+    <parent link="tool0"/>
 <!--    <origin xyz="-0.158 -0.158 0.123" rpy="0.0 ${radians(90)} ${radians(-135)}"/>-->
-    <origin xyz="-0.149 ${-0.149 - 0.005} 0.123" rpy="0.0 ${radians(-90)} ${radians(-135)}"/>
+    <origin xyz="-0.149 ${-0.149 - 0.005} 0.083" rpy="0.0 ${radians(-90)} ${radians(-135)}"/>
 <!--    <parent link="ee"/>-->
 <!--    <origin xyz="${-0.186 - 0.038} 0.0 ${0.08325}" rpy="0.0 ${radians(90)} 0.0"/>-->

Commit message: Updated application to specify camera frame relative robot controller-published flange frame

File: urdf/workcell.xacro (robot description, xacro)
@@ -5,5 +5,4 @@
   <xacro:include filename="$(find snp_automate_2023)/urdf/ros2_control.xacro"/>
   <xacro:snp_ros2_control name="snp_ros2_control" prefix=""/>
-  <xacro:property name="dt_flange_width" value="0.040"/>
   <!-- Add World -->
   <material name="light_gray">
@@ -66,9 +65,10 @@
   </joint>
   <!-- Create a frame representing the robot tool flange (behind the teach tool and nominal tool0 frame) for IKFast -->
-  <link name="tool_flange"/>
-  <joint name="tool0_to_tool_flange" type="fixed">
+  <!-- TODO Remove after updating to official version of HC10 support package -->
+  <link name="flange"/>
+  <joint name="tool0_to_flange" type="fixed">
     <parent link="tool0"/>
-    <child link="tool_flange"/>
-    <origin xyz="0.0 0.0 ${-dt_flange_width}" rpy="0 0 0"/>
+    <child link="flange"/>
+    <origin xyz="0 0 0" rpy="0 ${radians(-90)} ${radians(-180)}"/>
   </joint>
   <!-- Add End Effector Components -->
@@ -162,17 +162,10 @@
     <xacro:property name="camera_cal" value="${load_yaml('$(find snp_automate_2023)/config/calibration.yaml')}" />
   </xacro:unless>
-  <link name="camera_color_optical_frame"/>
+  <link name="camera_frame"/>
   <joint name="tool0_to_camera" type="fixed">
-    <parent link="tool0"/>
-    <child link="camera_color_optical_frame"/>
+    <parent link="flange"/>
+    <child link="camera_frame"/>
     <origin xyz="${camera_cal['camera_mount_to_camera_pos']['x']} ${camera_cal['camera_mount_to_camera_pos']['y']} ${camera_cal['camera_mount_to_camera_pos']['z']}"
             rpy="${camera_cal['camera_mount_to_camera_rpy']['x']} ${camera_cal['camera_mount_to_camera_rpy']['y']} ${camera_cal['camera_mount_to_camera_rpy']['z']}" />
-  </joint>
-  <link name="cal_target_frame"/>
-  <joint name="target_mount_to_target" type="fixed">
-    <parent link="base_link"/>
-    <child link="cal_target_frame"/>
-    <origin xyz="${camera_cal['target_mount_to_target_pos']['x']} ${camera_cal['target_mount_to_target_pos']['y']} ${camera_cal['target_mount_to_target_pos']['z']}"
-            rpy="${camera_cal['target_mount_to_target_rpy']['x']} ${camera_cal['target_mount_to_target_rpy']['y']} ${camera_cal['target_mount_to_target_rpy']['z']}" />
   </joint>
   <!-- Add TCP -->
@@ -190,7 +183,7 @@
   </link>
   <joint name="sand_tcp_joint" type="fixed">
-    <parent link="tool_flange"/>
+    <parent link="tool0"/>
 <!--    <origin xyz="-0.158 -0.158 0.123" rpy="0.0 ${radians(90)} ${radians(-135)}"/>-->
-    <origin xyz="-0.149 ${-0.149 - 0.005} 0.123" rpy="0.0 ${radians(-90)} ${radians(-135)}"/>
+    <origin xyz="-0.149 ${-0.149 - 0.005} 0.083" rpy="0.0 ${radians(-90)} ${radians(-135)}"/>
 <!--    <parent link="ee"/>-->
 <!--    <origin xyz="${-0.186 - 0.038} 0.0 ${0.08325}" rpy="0.0 ${radians(90)} 0.0"/>-->
